File: ESP12_pcb.kicad_pcb (KiCad board)
At the start: 2 copper layers, 0 parts

Commit message: Finished power components
Parts:
- added 12V1: TEST, Measurement_Points:Measurement_Point_Round-SMD-Pad_Small, F.Cu at (113.0, 87.6)
- added 3V3: TEST, Measurement_Points:Measurement_Point_Round-SMD-Pad_Small, F.Cu at (127.0, 95.2)
- added 5V1: TEST, Measurement_Points:Measurement_Point_Round-SMD-Pad_Small, F.Cu at (113.0, 94.0)
- added C1: 10uF, papayagroup:C_3528, F.Cu at (115.6, 83.8)
- added C2: 10uF, papayagroup:C_3528, F.Cu at (128.3, 88.9)
- added C3: 10uF, Capacitors_SMD:C_0603_HandSoldering, F.Cu at (118.1, 95.8)
- added C4: 0,1uF, Capacitors_SMD:C_0603_HandSoldering, F.Cu at (118.1, 97.8)
- added C5: 2.2uF, Capacitors_SMD:C_0603_HandSoldering, F.Cu at (115.6, 111.8)
- added C6: 100uF, Capacitors_SMD:C_0805_HandSoldering, F.Cu at (118.1, 111.8)
- added CON1: ZX62D1-B-5PA(30), papayagroup:USB-micro-B_Hirose, F.Cu at (100.3, 104.1)
- added D1: MBR120VLSFT3G, Diodes_SMD:D_SOD-123F, F.Cu at (115.6, 90.2)
- added D2: MBR120VLSFT3G, Diodes_SMD:D_SOD-123F, F.Cu at (132.1, 96.5)
- added F1: 0603L100SLYR, Resistors_SMD:R_0603_HandSoldering, F.Cu at (110.5, 91.4)
- added J1: CONN_01X02, Pin_Headers:Pin_Header_Straight_1x02_Pitch2.54mm, F.Cu at (133.1, 85.9)
- added J2: CONN_01X02_FEMALE, Connectors:bornier2, F.Cu at (104.1, 91.4)
- added L1: 6.8uH, papayagroup:L_bourns, F.Cu at (128.3, 105.4)
- added LBO1: TEST, Measurement_Points:Measurement_Point_Round-SMD-Pad_Small, F.Cu at (125.0, 114.3)
- added Q1: IRLML9301TRPBF, TO_SOT_Packages_SMD:SOT-23, F.Cu at (110.5, 83.8)
- added Q2: IRLML9301TRPBF, TO_SOT_Packages_SMD:SOT-23, F.Cu at (132.1, 92.7)
- added R1: 340k, Resistors_SMD:R_0603_HandSoldering, F.Cu at (123.2, 96.5)
- added R2: 2M, Resistors_SMD:R_0603_HandSoldering, F.Cu at (111.8, 101.6)
- added R3: 390k, Resistors_SMD:R_0603_HandSoldering, F.Cu at (109.2, 101.6)
- added R4: 1,87M, Resistors_SMD:R_0603_HandSoldering, F.Cu at (115.6, 108.0)
- added R5: 200k, Resistors_SMD:R_0603_HandSoldering, F.Cu at (110.5, 108.0)
- added R6: 1M, Resistors_SMD:R_0603_HandSoldering, F.Cu at (120.7, 111.8)
- added REF**: Drill_3mm, papayagroup:Drill_3mm, F.Cu at (108.0, 111.8)
- added REF**: Drill_3mm, papayagroup:Drill_3mm, F.Cu at (129.0, 83.3)
- added REF**: Drill_3mm, papayagroup:Drill_3mm, F.Cu at (102.6, 83.3)
- added U1: LD1117DT33TR, TO_SOT_Packages_SMD:TO-252-2Lead, F.Cu at (121.9, 83.8)
- added U2: TPS61090, papayagroup:QFN65P400X400X100-17N, F.Cu at (116.8, 102.9)
- added VDD1: TEST, Measurement_Points:Measurement_Point_Round-SMD-Pad_Small, F.Cu at (120.7, 106.7)
Routing:
- net +3V3: track 0.00 -> 42.8 mm
- net /LBO: track 0.00 -> 18.7 mm, vias 0 -> 2
- net VDD: track 0.00 -> 18.3 mm
- net /TPEN: track 0.00 -> 16.0 mm, vias 0 -> 2
- net +12V: track 0.00 -> 15.9 mm
- net Net-(L1-Pad2): track 0.00 -> 15.2 mm
- net Net-(CON1-Pad1): track 0.00 -> 14.4 mm
- net GND: track 0.00 -> 11.2 mm
- net Net-(J2-Pad2): track 0.00 -> 10.4 mm
- net +5V: track 0.00 -> 7.98 mm
- net Net-(R2-Pad2): track 0.00 -> 7.76 mm
- net Net-(R4-Pad2): track 0.00 -> 7.40 mm
- net Net-(J1-Pad2): track 0.00 -> 4.32 mm
- net +BATT: track 0.00 -> 4.25 mm
- added copper zone on B.Cu, net GND
- added copper zone on F.Cu, net GND
Other:
- board outline added: 36.8 x 36.8 mm
