File: ESP12_pcb.sch (KiCad schematic (older format))
At the start: 29 parts, among them CON1 ZX62D1-B-5PA(30), J1 CONN_01X02, J2 CONN_01X02_FEMALE, Q1 IRLML9301TRPBF, Q2 IRLML9301TRPBF, U1 LD1117DT33TR, U2 TPS61090

Commit message: Version V0.1 sended to fabrication
Parts:
- removed 12V1, 3V3, 5V1, GND1, LBO1, VDD1: TEST, Measurement_Points:Measurement_Point_Round-SMD-Pad_Small, symbol TEST
- removed C1, C2: 10uF, papayagroup:C_3528, symbol CP1
- removed CON1: ZX62D1-B-5PA(30), papayagroup:USB-micro-B_Hirose, symbol ZX62D1-B-5PA(30)
- removed D1, D2: MBR120VLSFT3G, Diodes_SMD:D_SOD-123F, symbol MBR120VLSFT3G
- removed F1: 0603L100SLYR, Resistors_SMD:R_0603_HandSoldering, symbol Polyfuse
- removed J2: CONN_01X02_FEMALE, Connectors:bornier2, symbol CONN_01X02_FEMALE
- removed Q1: IRLML9301TRPBF, TO_SOT_Packages_SMD:SOT-23, symbol Q_PMOS_GSD
- removed U1: LD1117DT33TR, TO_SOT_Packages_SMD:TO-252-2Lead, symbol LD1117DT33TR
- removed U2: TPS61090, papayagroup:QFN65P400X400X100-17N, symbol TPS61090
- added C1: 10uF, Capacitors_SMD:C_0603_HandSoldering, symbol C
- added C2: 100nF, Capacitors_SMD:C_0603_HandSoldering, symbol C
- added J3: Conn_02x04_Odd_Even, Pin_Headers:Pin_Header_Straight_2x04_Pitch2.54mm, symbol Conn_02x04_Odd_Even
- added R10, R11, R12: 10k, Resistors_SMD:R_0603_HandSoldering, symbol R
- added R5: 2M, Resistors_SMD:R_0603_HandSoldering, symbol R
- added R6: 12M, Resistors_SMD:R_0603_HandSoldering, symbol R
- added R7: 0, Resistors_SMD:R_0603_HandSoldering, symbol R
- added SW1: SW_Push, papayagroup:button_4pin, symbol SW_Push
- added TP1: bat, Measurement_Points:Measurement_Point_Round-SMD-Pad_Small, symbol TEST
- added TP2: vdd, Measurement_Points:Measurement_Point_Round-SMD-Pad_Small, symbol TEST
- added TP3: LBO, Measurement_Points:Measurement_Point_Round-SMD-Pad_Small, symbol TEST
- added U1: TPS61030PWR, papayagroup:R-PDSO-16, symbol TPS61030PWR
- C6: footprint Capacitors_SMD:C_0805_HandSoldering -> papayagroup:smd_5_5.4
- L1: footprint papayagroup:L_bourns -> papayagroup:smd_L_4532
- R4: value 1,87M -> 2M
- R8: renamed from R5; value 200k -> 220k
- renumbered R6 to R9
Connections:
- net +BATT: now also C3.1, C4.1, L1.1, R1.1, R2.1, TP1.1, U1.6 (VBAT)
- net GND: now also C1.2, C2.2, J3.1 (Pin_1), SW1.2, U1.11 (GND), U1.3 (PGND), U1.4 (PGND), U1.5 (PGND), U1.8 (SYNC)
- net LBO: now also J3.3 (Pin_3), TP3.1, U1.10 (LBO)
- net TPEN: now also U1.9 (EN)
- net VDD: now also C2.1, J3.8 (Pin_8), R10.1, R11.1, R12.1, TP2.1, U1.13 (VOUT), U1.14 (VOUT), U1.15 (VOUT)
- net at L1.2: now also U1.1 (SW), U1.2 (SW)
- net at R2.2, R3.1: now also U1.7 (LBI)
- net at R4.2: now also R5.1; no longer R8.1
- new net: R5.2, R6.1, R7.1
- new net CH_PD: J3.4 (Pin_4), R11.2
- new net FB: R6.2, R7.2, R8.1, U1.12 (FB)
- new net FLASH: J3.5 (Pin_5), R12.2
- new net RST: C1.1, J3.6 (Pin_6), R10.2, SW1.1
- no-connect marks 0 -> 3
Other:
- note added: "ESP01 Config"
- note added: "Power flags"
- note added: "Power step up"
- note added: "R7 = 0omhs => Vout = 5V\nR7 = open => Vout = 3.3V"
- note added: "Vout setup"
- note removed: "Vo = 5v -> R4 = 1,8M\nVo = 3.3V -> R4 = 13M"
- moved on the sheet: C3, C4, C5, C6, J1, L1, Q2, R1, R2, R3, R8, R9
